File: hardware/epaper-breakout/epaper-breakout.sch (KiCad schematic (older format))
At the start: 90 parts, among them J1 XF2M-3315-1A, J2 C10418, J3 Conn_02x06_Counter_Clockwise, J4 ED060SC4, J5 Conn_01x01_Male, J6 Conn_01x01_Male, Q1 AO3401A, Q2 AO3401A, Q3 MMBT3904, Q4 MMBT3904, Q5 AO3401A, Q6 MMBT3904, U1 MCP1700-3302E_SOT23, U10 ED060SC7, U11 TP4056, U12 CH340C, U2 LT1945, U3 LT1945, U4 XC6206PxxxMR, U5 ESP32-WROVER, U6 ED060XC5, U7 LM358, U8 74HC4094-normal, U9 MCP9700AT-ETT

Commit message: Merge vroland master branch
Parts:
- removed C1, C6: 4.7uF, Capacitor_SMD:C_0603_1608Metric, symbol Device:CP
- removed J3: Conn_02x06_Counter_Clockwise, Connector_PinHeader_2.54mm:PinHeader_2x06_P2.54mm_Vertical, symbol Connector_Generic:Conn_02x06_Counter_Clockwise
- removed J5, J6: Conn_01x01_Male, Connector_PinHeader_2.54mm:PinHeader_1x01_P2.54mm_Vertical, symbol Connector:Conn_01x01_Male
- removed JP_TEMP1: Jumper, Jumper:SolderJumper-2_P1.3mm_Bridged2Bar_RoundedPad1.0x1.5mm, symbol Device:Jumper
- removed L3, L4: 22uH, Inductor_SMD:L_6.3x6.3_H3, symbol Device:L
- removed Q1, Q2, Q5: AO3401A, Package_TO_SOT_SMD:SOT-23, symbol Transistor_FET:AO3401A
- removed Q6: MMBT3904, Package_TO_SOT_SMD:SOT-23, symbol Transistor_BJT:MMBT3904
- removed R12: 1k, Resistor_SMD:R_0805_2012Metric, symbol Device:R
- removed R17: 27k, Resistor_SMD:R_0805_2012Metric, symbol Device:R
- removed RV1: 200k, epaper-breakout:EVM3ESX50B25, symbol Device:R_POT
- removed TP1: TestPoint_Probe, TestPoint:TestPoint_Pad_D1.0mm, symbol Connector:TestPoint_Probe
- removed U10: ED060SC7, epaper-breakout:AXT334124, symbol epd_breakout:ED060SC7
- removed U2, U3: LT1945, Package_SO:MSOP-10_3x3mm_P0.5mm, symbol Regulator_Switching:LT1945
- removed U7: LM358, Package_SO:SOP-8_3.76x4.96mm_P1.27mm, symbol Amplifier_Operational:LM358
- removed U8: 74HC4094-normal, Package_SO:SOIC-16_3.9x9.9mm_P1.27mm, symbol 74HC4094:74HC4094-normal
- removed U9: MCP9700AT-ETT, Package_TO_SOT_SMD:SOT-23, symbol Sensor_Temperature:MCP9700AT-ETT
- added C1, C24, C26, C28, C31: 4.7uF, Capacitor_SMD:C_0805_2012Metric, symbol Device:C
- added C25: 10nF, Capacitor_SMD:C_0805_2012Metric, symbol Device:C
- added C27, C33: 2.2uF, Capacitor_SMD:C_0805_2012Metric, symbol Device:C
- added C29, C30, C39, C40: 100nF, Capacitor_SMD:C_0805_2012Metric, symbol Device:C
- added C32: 10uF, Capacitor_SMD:C_0805_2012Metric, symbol Device:C
- added C34, C36: 1uF/50V, Capacitor_SMD:C_1206_3216Metric, symbol Device:C
- added C35, C37, C38: 1uF/25V, Capacitor_SMD:C_0805_2012Metric, symbol Device:C
- added C6: 22uF, Capacitor_SMD:C_0805_2012Metric, symbol Device:C
- added J3: Conn_02x05_Counter_Clockwise, Connector_PinHeader_2.54mm:PinHeader_2x05_P2.54mm_Vertical, symbol Connector_Generic:Conn_02x05_Counter_Clockwise
- added J5: Conn_01x02_Female, Connector_PinHeader_2.54mm:PinHeader_1x02_P2.54mm_Vertical, symbol Connector:Conn_01x02_Female
- added J7: Conn_01x12, Connector_PinHeader_2.54mm:PinHeader_2x06_P2.54mm_Vertical, symbol Connector_Generic:Conn_01x12
- added R23: 1M, Resistor_SMD:R_0603_1608Metric, symbol Device:R
- added R24: 47.5k, Resistor_SMD:R_0603_1608Metric, symbol Device:R
- added R25: 10k, Resistor_SMD:R_0603_1608Metric, symbol Device:R
- added R26, R27, R28, R29: 47k, Resistor_SMD:R_0603_1608Metric, symbol Device:R
- added R30: 100k, Resistor_SMD:R_0603_1608Metric, symbol Device:R
- added TH1: 10k/3380K, Resistor_SMD:R_0603_1608Metric, symbol Device:Thermistor_NTC
- added TP1: +22V, TestPoint:TestPoint_Pad_D2.5mm, symbol Connector:TestPoint
- added TP2: -15V, TestPoint:TestPoint_Pad_D2.5mm, symbol Connector:TestPoint
- added TP3: -20V, TestPoint:TestPoint_Pad_D2.5mm, symbol Connector:TestPoint
- added TP4: +15V, TestPoint:TestPoint_Pad_D2.5mm, symbol Connector:TestPoint
- added TP5: VCOM, TestPoint:TestPoint_Pad_D2.5mm, symbol Connector:TestPoint
- added U2: PCA9535PW, Package_SO:TSSOP-24_4.4x7.8mm_P0.65mm, symbol Interface_Expansion:PCA9555PW
- added U3: TPS651851RSLR, tps65185:TPS651851RSLR, symbol TPS651851RSLR:TPS651851RSLR
- added U7: TPS2113APW, epaper-breakout:TPS2113APW, symbol epd_breakout:TPS2113APW
- C10: value 4.7pF -> 22uF; footprint Capacitor_SMD:C_0603_1608Metric -> Capacitor_SMD:C_0805_2012Metric; LCSC C1669 -> C45783
- C11, C8: value 100pF -> 4.7uF; footprint Capacitor_SMD:C_0603_1608Metric -> Capacitor_SMD:C_0805_2012Metric; LCSC C14858 -> C1779
- C12, C9: value 1uF -> 10uF; footprint Capacitor_SMD:C_0603_1608Metric -> Capacitor_SMD:C_0805_2012Metric; LCSC C15849 -> C15850
- C13, C14, C18: footprint Capacitor_SMD:C_0603_1608Metric -> Capacitor_SMD:C_0805_2012Metric; LCSC C15849 -> C28323
- C15: value 0.1uF -> 100nF; footprint Capacitor_SMD:C_0603_1608Metric -> Capacitor_SMD:C_0805_2012Metric; LCSC C1588 -> C49678
- C16, C22, C23: value 0.1uF -> 100nF; footprint Capacitor_SMD:C_0603_1608Metric -> Capacitor_SMD:C_0805_2012Metric; LCSC C14663 -> C49678
- C19: value 1uF -> 10uF; footprint Capacitor_SMD:C_0603_1608Metric -> Capacitor_SMD:C_0805_2012Metric; LCSC C15849 -> C19702
- C2, C3: footprint Capacitor_SMD:C_0603_1608Metric -> Capacitor_SMD:C_0805_2012Metric; LCSC C19702 -> C15850
- C20: value 1uF -> 10nF; footprint Capacitor_SMD:C_0603_1608Metric -> Capacitor_SMD:C_0805_2012Metric; LCSC C15849 -> C1710
- C21: value 10uF -> 100nF; footprint Capacitor_SMD:C_0603_1608Metric -> Capacitor_SMD:C_0805_2012Metric; LCSC C19702 -> C49678
- C4, C7: value 0.1uF -> 4.7uF; footprint Capacitor_SMD:C_0603_1608Metric -> Capacitor_SMD:C_0805_2012Metric; LCSC C14663 -> C1779
- C5: value 4.7pF -> 4.7uF; footprint Capacitor_SMD:C_0603_1608Metric -> Capacitor_SMD:C_0805_2012Metric; LCSC C1669 -> C1779
- J4: LCSC C92280 -> C519255
- L1: value 22uH -> 4.7uH; footprint Inductor_SMD:L_6.3x6.3_H3 -> Inductor_SMD:L_Taiyo-Yuden_NR-50xx_HandSoldering; LCSC C206321 -> C222947
- L2: value 22uH -> 2.2uH; footprint Inductor_SMD:L_6.3x6.3_H3 -> Inductor_SMD:L_Taiyo-Yuden_NR-40xx_HandSoldering; LCSC C206321 -> C92959
- R1, R10, R11, R13, R15: footprint Resistor_SMD:R_0805_2012Metric -> Resistor_SMD:R_0603_1608Metric; LCSC C17414 -> C25804
- R14: value 390k -> 10k; footprint Resistor_SMD:R_0805_2012Metric -> Resistor_SMD:R_0603_1608Metric; LCSC C17656 -> C25804
- R16: value 300k -> 10k; footprint Resistor_SMD:R_0805_2012Metric -> Resistor_SMD:R_0603_1608Metric; LCSC C17616 -> C25804
- R18: value 110k -> 43k; footprint Resistor_SMD:R_0805_2012Metric -> Resistor_SMD:R_0603_1608Metric; LCSC C17422 -> C23172
- R19: value 10k -> 1M; footprint Resistor_SMD:R_0805_2012Metric -> Resistor_SMD:R_0603_1608Metric; LCSC C17414 -> C22935
- R2: value 100k -> 400; footprint Resistor_SMD:R_0805_2012Metric -> Resistor_SMD:R_0603_1608Metric; LCSC C17407 -> C23151
- R20: value 10k -> 52.3k; footprint Resistor_SMD:R_0805_2012Metric -> Resistor_SMD:R_0603_1608Metric; LCSC C17414 -> C23196
- R21: footprint Resistor_SMD:R_0805_2012Metric -> Resistor_SMD:R_0603_1608Metric; LCSC C17797 -> C25822
- R22: footprint Resistor_SMD:R_0805_2012Metric -> Resistor_SMD:R_0603_1608Metric; LCSC C17470 -> C22807
- R3, R8: footprint Resistor_SMD:R_0805_2012Metric -> Resistor_SMD:R_0603_1608Metric; LCSC C17513 -> C21190
- R4: value 2M -> 10k; footprint Resistor_SMD:R_0805_2012Metric -> Resistor_SMD:R_0603_1608Metric; LCSC C26112 -> C25804
- R5: value 120k -> 0; footprint Resistor_SMD:R_0805_2012Metric -> Resistor_SMD:R_0603_1608Metric; LCSC C17436 -> (none)
- R6: value 560k -> 10k; footprint Resistor_SMD:R_0805_2012Metric -> Resistor_SMD:R_0603_1608Metric; LCSC C15785 -> C25804
- R7: value 39k -> 100k; footprint Resistor_SMD:R_0805_2012Metric -> Resistor_SMD:R_0603_1608Metric; LCSC C25826 -> C25803
- R9: footprint Resistor_SMD:R_0805_2012Metric -> Resistor_SMD:R_0603_1608Metric; LCSC C17772 -> C23212
- U6: LCSC (none) -> C528053
Connections:
- net labels added: SCL, SDA, TPS_PWRUP, TPS_PWR_GOOD, TPS_VCOM_CTRL, TPS_WAKEUP, TPS_nINT, USB_D+, USB_D-, VNEG_IN, ~GPIO_INTR
- net labels removed: A1, CTRL+15V, CTRL+22V, CTRL-15V, CTRL-20V, SMPS_CTRL, V_TEMP
- wire segments 498 -> 514
Other:
- note added: "Close to EPD connector"
- note removed: "Epaper Common Voltage"
- note removed: "SMPS Power +22V, -20V"
- note removed: "Unused opamp neutralizer"
- moved on the sheet: C13, C14, C15, C16, C17, C18, C2, C22, C23, C3, D10, D8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
