File: hardware/extension-9_40_to_34_6inch/extension-cable.kicad_sch (KiCad schematic)
At the start: 8 parts, among them J1 XF2M-3315-1A, U1 ED060XC5, U2 ED078KH6, U3 ED060XC5

Commit message: Add PCB tester with LEDs & MicroSD
Parts:
- J1: LCSC C231420 -> C597986
Changed lines of the file:
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@@
       (effects (font (size 1.524 1.524)))
     )
-    (property "LCSC" "C231420" (at 46.355 49.53 0)
+    (property "LCSC" "C597986" (at 46.355 49.53 0)
       (effects (font (size 1.27 1.27)) hide)
     )
